Commit message: 002

File: src/double_invert_pendulum_description/robot/visual/double_invert_pendulum.xacro (robot description, xacro)
@@ -8,5 +8,5 @@
     <link name="world"/>
     <!-- FIXED JOINT (Base stuck to ground - no cart movement) -->
-    <joint name="cart_joint" type="fixed">
+    <joint name="base" type="fixed">
         <parent link="world"/>
         <child link="base_link"/>

Commit message: 001

File: src/double_invert_pendulum_description/robot/visual/double_invert_pendulum.xacro (robot description, xacro)
@@ -13,17 +13,14 @@
         <origin xyz="0 0 0" rpy="0 0 0"/>  <!-- Base origin at ground level -->
     </joint>
-    <!-- BASE LINK (CART) -->
+    <!-- BASE LINK -->
     <link name="base_link">
-        <inertial>
+        <!--
+          FIX: Using macro to calculate inertia from the mass variable
+          in pendulum_params.xacro and the collision box size.
+        -->
+        <xacro:inertial_box mass="${mass_base}" x="0.25" y="0.15" z="0.18">
+            <!-- Origin from original URDF -->
             <origin xyz="4.35011143188239E-06 -4.26974202710915E-05 0.0926893522450359" rpy="0 0 0" />
-            <mass value="${mass_base}" />
-            <inertia
-                ixx="0.00149406454043322"
-                ixy="4.12697804108289E-09"
-                ixz="-7.65282756367958E-08"
-                iyy="0.00140648625642533"
-                iyz="8.80770910699998E-10"
-                izz="0.000630646344660402" />
-        </inertial>
+        </xacro:inertial_box>
         <visual>
             <origin xyz="0 0 0" rpy="0 0 0" />
@@ -34,6 +31,4 @@
         </visual>
         <collision>
-            <!-- Using box primitive for better collision physics -->
-            <!-- Box positioned to match the base geometry -->
             <origin xyz="0 0 0.09" rpy="0 0 0" />
             <geometry>
@@ -42,25 +37,23 @@
         </collision>
     </link>
-    <!-- REVOLUTE LINK -->
-    <joint name="revolute_joint" type="revolute">
+    <!-- REVOLUTE LINK (CONTINUOUS - unlimited rotation) -->
+    <joint name="revolute_joint" type="continuous">
         <parent link="base_link"/>
         <child link="revolute_Link"/>
         <origin xyz="${revolute_joint_x} ${revolute_joint_y} ${revolute_joint_z}" rpy="0 0 0"/>
         <axis xyz="0 0 1"/>
-        <limit effort="${joint_effort}" velocity="${joint_velocity}" lower="${joint_lower_limit}" upper="${joint_upper_limit}"/>
+        <limit effort="${joint_effort}" velocity="${joint_velocity}"/>
         <dynamics damping="${revolute_joint_damping}" friction="${revolute_joint_friction}"/>
     </joint>
     <link name="revolute_Link">
-        <inertial>
-            <origin xyz="-0.0175370700578145 -0.00016469410235089 0.00111078231813694" rpy="0 0 0" />
-            <mass value="${mass_revolute}" />
-            <inertia
-                ixx="5.58988467068262E-05"
-                ixy="-2.47845250293903E-09"
-                ixz="-6.15261336732486E-09"
-                iyy="8.47733759009359E-05"
-                iyz="4.85611321474861E-09"
-                izz="0.000107267938774701" />
-        </inertial>
+        <!--
+          FIX: Using inertial_cylinder macro to calculate inertia based on
+          the '${mass_revolute}' variable from pendulum_params.xacro.
+          This replaces the hard-coded PDF values.
+        -->
+        <xacro:inertial_cylinder mass="${mass_revolute}" length="0.05" radius="0.03">
+             <!-- Origin from SolidWorks PDF, converted to meters -->
+            <origin xyz="-0.0393104703 -0.0011200394 -0.0049654099" rpy="0 0 0" />
+        </xacro:inertial_cylinder>
         <visual>
             <origin xyz="0 0 0" rpy="0 0 0" />
@@ -71,5 +64,4 @@
         </visual>
         <collision>
-            <!-- Using cylinder primitive for revolute joint housing -->
             <origin xyz="0 0 0" rpy="0 0 0" />
             <geometry>
@@ -88,15 +80,12 @@
     </joint>
     <link name="first_pendulum_link">
-        <inertial>
-            <origin xyz="-1.00551614541671E-07 -0.0646186151454772 -0.00362087479361183" rpy="0 0 0" />
-            <mass value="${mass_pendulum1}" />
-            <inertia
-                ixx="0.000174588068807012"
-                ixy="-2.95045790870356E-10"
-                ixz="2.21709158691471E-11"
-                iyy="6.96835664909535E-06"
-                iyz="5.24978381703527E-07"
-                izz="0.000169216758156749" />
-        </inertial>
+        <!--
+          FIX: Using inertial_box macro to calculate inertia based on
+          the '${mass_pendulum1}' variable from pendulum_params.xacro.
+        -->
+        <xacro:inertial_box mass="${mass_pendulum1}" x="0.02" y="0.14" z="0.02">
+            <!-- Origin from SolidWorks PDF, converted to meters -->
+            <origin xyz="-0.0000001372 -0.0878320187 0.0001351167" rpy="0 0 0" />
+        </xacro:inertial_box>
         <visual>
             <origin xyz="0 0 0" rpy="0 0 0" />
@@ -107,5 +96,4 @@
         </visual>
         <collision>
-            <!-- Using box primitive for first pendulum rod -->
             <origin xyz="0 -0.065 0" rpy="0 0 0" />
             <geometry>
@@ -124,15 +112,12 @@
     </joint>
     <link name="second_pendulum_link">
-        <inertial>
-            <origin xyz="-2.8765755728709E-06 -0.0299439674255459 0.00119447713150889" rpy="0 0 0" />
-            <mass value="${mass_pendulum2}" />
-            <inertia
-                ixx="1.8911424822564E-06"
-                ixy="-9.8432286079085E-12"
-                ixz="2.35767361175274E-10"
-                iyy="2.84550526022121E-07"
-                iyz="3.87915762114474E-08"
-                izz="2.05641965585819E-06" />
-        </inertial>
+        <!--
+          FIX: Using inertial_box macro to calculate inertia based on
+          the '${mass_pendulum2}' variable from pendulum_params.xacro.
+        -->
+        <xacro:inertial_box mass="${mass_pendulum2}" x="0.015" y="0.06" z="0.015">
+            <!-- Origin from SolidWorks PDF, converted to meters -->
+            <origin xyz="-0.0000028766 -0.0299439674 0.001944771" rpy="0 0 0" />
+        </xacro:inertial_box>
         <visual>
             <origin xyz="0 0 0" rpy="0 0 0" />
@@ -143,5 +128,4 @@
         </visual>
         <collision>
-            <!-- Using box primitive for second pendulum rod -->
             <origin xyz="0 -0.03 0" rpy="0 0 0" />
             <geometry>

File: src/double_invert_pendulum_description/robot/visual/gazebo_full.xacro (robot description, xacro)
@@ -24,5 +24,5 @@
       </command_interface>
       <state_interface name="position">
-        <param name="initial_value">0.0</param>
+        <param name="initial_value"> 0.0 </param>
       </state_interface>
       <state_interface name="velocity"/>

File: src/double_invert_pendulum_description/robot/visual/pendulum_params.xacro (robot description, xacro)
@@ -13,22 +13,24 @@
     <xacro:property name="pendulum2_joint_y" value="-0.1432"/>
     <xacro:property name="pendulum2_joint_z" value="0.0095"/>
-    <!-- Masses from original URDF -->
-    <xacro:property name="mass_base" value="0.951310569253784"/>
-    <xacro:property name="mass_revolute" value="0.216240646404497"/>
-    <xacro:property name="mass_pendulum1" value="0.0997302210483473"/>
-    <xacro:property name="mass_pendulum2" value="0.00680601326910171"/>
+    <!--
+      Masses updated to match SolidWorks PDF reports (converted g -> kg)
+    -->
+    <xacro:property name="mass_base" value="0.5"/> <!-- Value from previous file, no PDF provided -->
+    <xacro:property name="mass_revolute" value="0.134003"/> <!-- 134.003 g -->
+    <xacro:property name="mass_pendulum1" value="0.050"/>    <!-- 50.0 g -->
+    <xacro:property name="mass_pendulum2" value="0.015"/>    <!-- 15.0 g -->
     <!-- Joint limits - converted from continuous to revolute -->
     <xacro:property name="joint_effort" value="100"/>
-    <xacro:property name="joint_velocity" value="10"/>
+    <xacro:property name="joint_velocity" value=" 50.0 "/>
     <xacro:property name="joint_lower_limit" value="${-PI}"/>
     <xacro:property name="joint_upper_limit" value="${PI}"/>
     <!-- Joint dynamics - Revolute Joint -->
-    <xacro:property name="revolute_joint_damping" value="0.1"/>
-    <xacro:property name="revolute_joint_friction" value="0.05"/>
+    <xacro:property name="revolute_joint_damping" value="0.001"/>
+    <xacro:property name="revolute_joint_friction" value="0.02"/>
     <!-- Joint dynamics - First Pendulum -->
-    <xacro:property name="first_pendulum_damping" value="0.01"/>
-    <xacro:property name="first_pendulum_friction" value="0.001"/>
+    <xacro:property name="first_pendulum_damping" value="0.001"/>
+    <xacro:property name="first_pendulum_friction" value="0.1"/>
     <!-- Joint dynamics - Second Pendulum -->
-    <xacro:property name="second_pendulum_damping" value="0.01"/>
-    <xacro:property name="second_pendulum_friction" value="0.001"/>
+    <xacro:property name="second_pendulum_damping" value="0.001"/>
+    <xacro:property name="second_pendulum_friction" value="0.1"/>
 </robot>

Commit message: 001

File: src/double_invert_pendulum_description/robot/visual/double_invert_pendulum.xacro (robot description, xacro)
@@ -66,5 +66,5 @@
         <origin xyz="${pendulum1_joint_x} ${pendulum1_joint_y} ${pendulum1_joint_z}" rpy="1.5708 0 -1.5708"/>
         <axis xyz="0 0 1"/>
-        <limit effort="${joint_effort}" velocity="${joint_velocity}" lower="${joint_lower_limit}" upper="${joint_upper_limit}"/>
+        <limit effort="100.0" velocity="100.0" lower="${joint_lower_limit}" upper="${joint_upper_limit}"/>
         <dynamics damping="${first_pendulum_damping}" friction="${first_pendulum_friction}"/>
     </joint>
@@ -93,5 +93,5 @@
         <origin xyz="${pendulum2_joint_x} ${pendulum2_joint_y} ${pendulum2_joint_z}" rpy="0 0 0"/>
         <axis xyz="0 0 1"/>
-        <limit effort="${joint_effort}" velocity="${joint_velocity}" lower="${joint_lower_limit}" upper="${joint_upper_limit}"/>
+        <limit effort="100.0" velocity="100.0" lower="${joint_lower_limit}" upper="${joint_upper_limit}"/>
         <dynamics damping="${second_pendulum_damping}" friction="${second_pendulum_friction}"/>
     </joint>

File: src/double_invert_pendulum_description/robot/visual/gazebo_full.xacro (robot description, xacro)
@@ -22,5 +22,5 @@
       </command_interface>
       <state_interface name="position">
-        <param name="initial_value">0</param>
+        <param name="initial_value">0.0</param>
       </state_interface>
       <state_interface name="velocity"/>

File: src/double_invert_pendulum_description/robot/visual/pendulum_params.xacro (robot description, xacro)
@@ -56,6 +56,6 @@
     <!-- ========================================== -->
     <!-- Joint effort and velocity limits -->
-    <xacro:property name="joint_effort" value="7.5"/>
-    <xacro:property name="joint_velocity" value="15.0"/>
+    <xacro:property name="joint_effort" value="100.0"/>
+    <xacro:property name="joint_velocity" value= "7.5"/>
     <xacro:property name="joint_lower_limit" value="${-2*PI}"/>
     <xacro:property name="joint_upper_limit" value="${2*PI}"/>
@@ -65,8 +65,8 @@
     <!-- First Pendulum Joint Dynamics - PASSIVE -->
     <xacro:property name="first_pendulum_damping" value="${c1_paper}"/>
-    <xacro:property name="first_pendulum_friction" value="0.001"/>
+    <xacro:property name="first_pendulum_friction" value="${c1_paper}"/>
     <!-- Second Pendulum Joint Dynamics - PASSIVE -->
     <xacro:property name="second_pendulum_damping" value="${c2_paper}"/>
-    <xacro:property name="second_pendulum_friction" value="0.001"/>
+    <xacro:property name="second_pendulum_friction" value="${c2_paper}"/>
     <!-- ========================================== -->
     <!-- COLLISION GEOMETRY PARAMETERS -->
